Commit message: refine

File: urdf/bottle64.urdf.xacro (robot description, xacro)
@@ -20,5 +20,5 @@
     <visual>
       <geometry>
-        <mesh filename="file:///home/xuxie/ROS/catkin_robotics/src/glove/post_tac_glove/urdf/meshes/bottle64.dae"/>
+        <mesh filename="file://$(arg meshdir)bottle64.dae"/>
       </geometry>
     </visual>
@@ -27,5 +27,5 @@
     <visual>
       <geometry>
-        <mesh filename="file:///home/xuxie/ROS/catkin_robotics/src/glove/post_tac_glove/urdf/meshes/bottle64_lid.dae"/>
+        <mesh filename="file://$(arg meshdir)bottle64_lid.dae"/>
       </geometry>
     </visual>

File: urdf/bottle68.urdf.xacro (robot description, xacro)
@@ -20,5 +20,5 @@
     <visual>
       <geometry>
-        <mesh filename="file:///home/xuxie/ROS/catkin_robotics/src/glove/post_tac_glove/urdf/meshes/bottle68.dae"/>
+        <mesh filename="file://$(arg meshdir)bottle68.dae"/>
       </geometry>
     </visual>
@@ -27,5 +27,5 @@
     <visual>
       <geometry>
-        <mesh filename="file:///home/xuxie/ROS/catkin_robotics/src/glove/post_tac_glove/urdf/meshes/bottle68_lid.dae"/>
+        <mesh filename="file://$(arg meshdir)bottle68_lid.dae"/>
       </geometry>
     </visual>

File: urdf/bottle69.urdf.xacro (robot description, xacro)
@@ -20,5 +20,5 @@
     <visual>
       <geometry>
-        <mesh filename="file:///home/xuxie/ROS/catkin_robotics/src/glove/post_tac_glove/urdf/meshes/bottle69.dae"/>
+        <mesh filename="file://$(arg meshdir)bottle69.dae"/>
       </geometry>
     </visual>
@@ -27,5 +27,5 @@
     <visual>
       <geometry>
-        <mesh filename="file:///home/xuxie/ROS/catkin_robotics/src/glove/post_tac_glove/urdf/meshes/bottle69_lid.dae"/>
+        <mesh filename="file://$(arg meshdir)bottle69_lid.dae"/>
       </geometry>
     </visual>
